Commit message: draft robot urdf v0.1

File: ros2/src/urdf_tutorial/urdf/carter/carter.urdf (robot description, URDF)
Before this commit: robot carter, 7 links, 6 joints
Links:
- removed link chassis_link
- added link base_link, mass 45.88; collision box size=.55 .40 .54; visual mesh filename=package://urdf_tutorial/meshes/carter/chassis.obj
- link left_wheel_link: geometry collision cylinder length=0.1 radius=0.240; visual mesh filename=package://urdf_tutorial/meshes/carter/side_wheel.obj
- link rear_pivot_link: geometry collision box size=.09 .08 .12; visual mesh filename=package://urdf_tutorial/meshes/carter/pivot.obj
- link rear_wheel_link: geometry collision cylinder length=0.04 radius=0.076; visual mesh filename=package://urdf_tutorial/meshes/carter/caster_wheel.obj
- link right_wheel_link: geometry collision cylinder length=0.1 radius=0.240; visual mesh filename=package://urdf_tutorial/meshes/carter/side_wheel.obj
Joints:
- joint com_joint: parent chassis_link -> base_link
- joint imu_joint: parent chassis_link -> base_link
- joint left_wheel: parent chassis_link -> base_link
- joint rear_pivot: parent chassis_link -> base_link
- joint right_wheel: parent chassis_link -> base_link

File: ros2/src/urdf_tutorial/urdf/test.urdf (robot description, URDF)
Before this commit: robot myfirst, 1 links, 0 joints
Links:
- added link chest, mass ${chest_mass}; collision cylinder length=${chest_length} radius=${chest_radius}; visual cylinder length=${chest_length} radius=${chest_radius}
- added link head, mass ${head_mass}; collision box size=${head_length} ${head_width} ${head_height}; visual box size=${head_length} ${head_width} ${head_height}
- added link left_front_wheel, mass ${wheel_mass}; collision cylinder length=${wheel_length} radius=${wheel_radius}; visual cylinder length=${wheel_length} radius=${wheel_radius}
- added link left_hand_base, mass ${hand_base_mass}; collision cylinder length=${hand_base_length} radius=${hand_base_radius}; visual cylinder length=${hand_base_length} radius=${hand_base_radius}
- added link left_lower_arm, mass ${lower_arm_mass}; collision box size=${lower_arm_length} ${lower_arm_width} ${lower_arm_height}; visual box size=${lower_arm_length} ${lower_arm_width} ${lower_arm_height}
- added link left_rear_wheel, mass ${wheel_mass}; collision cylinder length=${wheel_length} radius=${wheel_radius}; visual cylinder length=${wheel_length} radius=${wheel_radius}
- added link left_shoulder, mass ${shoulder_mass}; collision cylinder length=${shoulder_length} radius=${shoulder_radius}; visual cylinder length=${shoulder_length} radius=${shoulder_radius}
- added link left_upper_arm, mass ${upper_arm_mass}; collision box size=${upper_arm_length} ${upper_arm_width} ${upper_arm_height}; visual box size=${upper_arm_length} ${upper_arm_width} ${upper_arm_height}
- added link neck, mass ${neck_mass}; collision cylinder length=${neck_length} radius=${neck_radius}; visual cylinder length=${neck_length} radius=${neck_radius}
- added link right_front_wheel, mass ${wheel_mass}; collision cylinder length=${wheel_length} radius=${wheel_radius}; visual cylinder length=${wheel_length} radius=${wheel_radius}
- added link right_hand_base, mass ${hand_base_mass}; collision cylinder length=${hand_base_length} radius=${hand_base_radius}; visual cylinder length=${hand_base_length} radius=${hand_base_radius}
- added link right_lower_arm, mass ${lower_arm_mass}; collision box size=${lower_arm_length} ${lower_arm_width} ${lower_arm_height}; visual box size=${lower_arm_length} ${lower_arm_width} ${lower_arm_height}
- added link right_rear_wheel, mass ${wheel_mass}; collision cylinder length=${wheel_length} radius=${wheel_radius}; visual cylinder length=${wheel_length} radius=${wheel_radius}
- added link right_shoulder, mass ${shoulder_mass}; collision cylinder length=${shoulder_length} radius=${shoulder_radius}; visual cylinder length=${shoulder_length} radius=${shoulder_radius}
- added link right_upper_arm, mass ${upper_arm_mass}; collision box size=${upper_arm_length} ${upper_arm_width} ${upper_arm_height}; visual box size=${upper_arm_length} ${upper_arm_width} ${upper_arm_height}
- added link waist, mass ${waist_mass}; collision cylinder length=${waist_length} radius=${waist_radius}; visual cylinder length=${waist_length} radius=${waist_radius}
- link base_link: mass None -> ${base_mass}; geometry collision box size=${base_length} ${base_width} ${base_height}; visual box size=${base_length} ${base_width} ${base_height}
Joints:
- added joint chest_joint: type continuous, parent waist, child chest, origin xyz=0 0 ${waist_length+chest_length/2} rpy=0 0 0
- added joint head_joint: type continuous, parent neck, child head, origin xyz=0 0 ${neck_length+head_height/2} rpy=0 0 0, axis 0 0 1
- added joint left_front_wheel_joint: type continuous, parent base_link, child left_front_wheel, origin xyz=${base_length/2+0.1} ${base_width/2+wheel_length/2+0.1} -${wheel_height_offset} rpy=0 0 0, axis 0 1 0
- added joint left_hand_base_joint: type continuous, parent left_lower_arm, child left_hand_base, origin xyz=0 ${lower_arm_width+hand_base_length/2} 0 rpy=0 0 0, axis 0 1 0
- added joint left_lower_arm_joint: type continuous, parent left_upper_arm, child left_lower_arm, origin xyz=0 ${upper_arm_width+lower_arm_length/2} 0 rpy=0 0 0, axis 0 0 1
- added joint left_rear_wheel_joint: type continuous, parent base_link, child left_rear_wheel, origin xyz=-${base_length/2+0.1} ${base_width/2+wheel_length/2+0.1} -${wheel_height_offset} rpy=0 0 0, axis 0 1 0
- added joint left_shoulder_joint: type continuous, parent chest, child left_shoulder, origin xyz=0 ${chest_radius+shoulder_length/2} ${chest_length/2-shoulder_radius} rpy=0 0 0, axis 0 1 0
- added joint left_upper_arm_joint: type continuous, parent left_shoulder, child left_upper_arm, origin xyz=0 ${shoulder_length/2+upper_arm_length/2} 0 rpy=0 0 0, axis 1 0 0
- added joint neck_joint: type fixed, parent chest, child neck, origin xyz=0 0 ${chest_length/2} rpy=0 0 0
- added joint right_front_wheel_joint: type continuous, parent base_link, child right_front_wheel, origin xyz=${base_length/2+0.1} -${base_width/2+wheel_length/2+0.1} -${wheel_height_offset} rpy=0 0 0, axis 0 1 0
- added joint right_hand_base_joint: type continuous, parent right_lower_arm, child right_hand_base, origin xyz=0 -${lower_arm_width+hand_base_length/2} 0 rpy=0 0 0, axis 0 1 0
- added joint right_lower_arm_joint: type continuous, parent right_upper_arm, child right_lower_arm, origin xyz=0 -${upper_arm_width+lower_arm_length/2} 0 rpy=0 0 0, axis 0 0 1
- added joint right_rear_wheel_joint: type continuous, parent base_link, child right_rear_wheel, origin xyz=-${base_length/2+0.1} -${base_width/2+wheel_length/2+0.1} -${wheel_height_offset} rpy=0 0 0, axis 0 1 0
- added joint right_shoulder_joint: type continuous, parent chest, child right_shoulder, origin xyz=0 -${chest_radius+shoulder_length/2} ${chest_length/2-shoulder_radius} rpy=0 0 0, axis 0 1 0
- added joint right_upper_arm_joint: type continuous, parent right_shoulder, child right_upper_arm, origin xyz=0 -${shoulder_length/2+upper_arm_length/2} 0 rpy=0 0 0, axis 1 0 0
- added joint waist_joint: type fixed, parent base_link, child waist, origin xyz=0 0 ${base_height/2} rpy=0 0 0
